Commit message: replaced the default simple_driving with the lidar version

File: simple_driving/resources/simplecar.urdf (robot description, URDF)
Before this commit: robot simplecar, 7 links, 6 joints
Links:
- added link lidar_link, mass 0.1; collision cylinder length=0.08 radius=0.04; visual cylinder length=0.08 radius=0.04
Joints:
- added joint base_to_lidar: type fixed, parent base_link, child lidar_link, origin xyz=0 0 0.25 rpy=0 0 0
