Commit message: things spawn mostly good :)
Co-authored-by: Copilot <copilot@github.com>

File: src/simple_driving/resources/simpleplane.urdf (robot description, URDF)
Before this commit: robot simpleplane, 1 links, 0 joints
Links:
- link base_link: geometry collision box size=10000 10000 0.01; visual box size=10000 10000 0.01
